File: Circuit/boneIO - relay board/boneIO - relay board.kicad_pcb (KiCad board)
At the start: 2 copper layers, 197 x 102 mm, 68 parts, among them J1 Screw_Terminal_01x04, J10 Screw_Terminal_01x04, J11 Screw_Terminal_01x04, J12 Screw_Terminal_01x04, J13 Screw_Terminal_01x04, J14 Conn_02x04_Odd_Even, J2 Screw_Terminal_01x04, J4 Screw_Terminal_01x04, J5 Screw_Terminal_01x04, J6 Screw_Terminal_01x04, J7 Screw_Terminal_01x04, J8 Screw_Terminal_01x04, J9 Screw_Terminal_01x04, K1 RM85-2011-35-1005, K10 RM85-2011-35-1005, K11 RM85-2011-35-1005, K12 RM85-2011-35-1005, K13 RM85-2011-35-1005, K14 RM85-2011-35-1005, K15 RM85-2011-35-1005, K16 RM85-2011-35-1005, K17 RM85-2011-35-1005, K18 RM85-2011-35-1005, K19 RM85-2011-35-1005, K2 RM85-2011-35-1005, K20 RM85-2011-35-1005, K21 RM85-2011-35-1005, K22 RM85-2011-35-1005, K23 RM85-2011-35-1005, K24 RM85-2011-35-1005, K3 RM85-2011-35-1005, K4 RM85-2011-35-1005, K5 RM85-2011-35-1005, K6 RM85-2011-35-1005, K7 RM85-2011-35-1005, K8 RM85-2011-35-1005, K9 RM85-2011-35-1005, SW1 SW_DIP_x03, SW2 SW_DIP_x03, SW3 SW_DIP_x03, U1 MCP9808_MSOP, U2 MCP23017_SS, U3 MCP23017_SS, U4 ULN2803A, U5 ULN2803A, U6 ULN2803A

Commit message: Revert "Zmiana Nazwy płytki"
This reverts commit 4cfb8962ad837d49dd7d8c96a90ff7a4eda2ea33.
Other:
- board text added: "Relay Board v0.2"
- board text removed: "relay board 24x16A v0.2"
Changed lines of the file:
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@@
       (effects (font (size 1 1) (thickness 0.15)))
     )
+    (fp_text user %R (at 1.27 3.81) (layer F.Fab)
+      (effects (font (size 1 1) (thickness 0.15)))
+    )
     (fp_line (start 0 -1.27) (end 3.81 -1.27) (layer F.Fab) (width 0.1))
     (fp_line (start 3.81 -1.27) (end 3.81 8.89) (layer F.Fab) (width 0.1))
@@
     (fp_line (start 4.35 9.4) (end 4.35 -1.8) (layer F.CrtYd) (width 0.05))
     (fp_line (start 4.35 -1.8) (end -1.8 -1.8) (layer F.CrtYd) (width 0.05))
-    (fp_text user %R (at 1.27 3.81) (layer F.Fab)
-      (effects (font (size 1 1) (thickness 0.15)))
-    )
     (pad 8 thru_hole oval (at 2.54 7.62 90) (size 1.7 1.7) (drill 1) (layers *.Cu *.Mask)
       (net 79 SDA))
@@
     (effects (font (size 1 1) (thickness 0.15)))
   )
-  (gr_text "relay board 24x16A v0.2" (at 302.96 317.538) (layer F.SilkS)
+  (gr_text "Relay Board v0.2\n\n" (at 302.34 318.018) (layer F.SilkS)
     (effects (font (size 0.8 0.8) (thickness 0.14)))
   )
