File: Circuit/boneIO - relay board/boneIO - relay board.sch (KiCad schematic (older format))
At the start: 68 parts, among them J1 Screw_Terminal_01x04, J10 Screw_Terminal_01x04, J11 Screw_Terminal_01x04, J12 Screw_Terminal_01x04, J13 Screw_Terminal_01x04, J14 Conn_02x04_Odd_Even, J2 Screw_Terminal_01x04, J3 Conn_02x04_Odd_Even, J4 Screw_Terminal_01x04, J5 Screw_Terminal_01x04, J6 Screw_Terminal_01x04, J7 Screw_Terminal_01x04, J8 Screw_Terminal_01x04, J9 Screw_Terminal_01x04, K1 RM85-2011-35-1005, K10 RM85-2011-35-1005, K11 RM85-2011-35-1005, K12 RM85-2011-35-1005, K13 RM85-2011-35-1005, K14 RM85-2011-35-1005, K15 RM85-2011-35-1005, K16 RM85-2011-35-1005, K17 RM85-2011-35-1005, K18 RM85-2011-35-1005, K19 RM85-2011-35-1005, K2 RM85-2011-35-1005, K20 RM85-2011-35-1005, K21 RM85-2011-35-1005, K22 RM85-2011-35-1005, K23 RM85-2011-35-1005, K24 RM85-2011-35-1005, K3 RM85-2011-35-1005, K4 RM85-2011-35-1005, K5 RM85-2011-35-1005, K6 RM85-2011-35-1005, K7 RM85-2011-35-1005, K8 RM85-2011-35-1005, K9 RM85-2011-35-1005, SW1 SW_DIP_x03, SW2 SW_DIP_x03, SW3 SW_DIP_x03, U1 MCP9808_MSOP, U2 MCP23017_SS, U3 MCP23017_SS, U4 ULN2803A, U5 ULN2803A, U6 ULN2803A

Commit message: Revert "Zmiana Nazwy płytki"
This reverts commit 4cfb8962ad837d49dd7d8c96a90ff7a4eda2ea33.
Other:
- note added: "boneIO - relay board v0.2"
- note removed: "boneIO - relay board 24x16A v0.2"
Changed lines of the file:
@@
 Text Notes 18650 2300 0    197  ~ 39
 MCP23017
-Text Notes 9200 1250 0    197  ~ 39
-boneIO - relay board 24x16A v0.2
+Text Notes 9600 1250 0    197  ~ 39
+boneIO - relay board v0.2
 Wire Wire Line
 	6750 100  6750 400
