File: Circuit/boneIO - input board/boneIO_input board.sch (KiCad schematic (older format))
At the start: 262 parts, among them J1 Screw_Terminal_01x08, J10 Screw_Terminal_01x08, J11 Screw_Terminal_01x08, J12 ZW_VCC, J13 ZW_GND, J14 INNY ZASILACZ, J15 BeagleBone_Black_Header, J16 BeagleBone_Black_Header, J2 Screw_Terminal_01x08, J3 Screw_Terminal_01x08, J4 Screw_Terminal_01x08, J5 Screw_Terminal_01x08, J6 Screw_Terminal_01x08, J7 Screw_Terminal_01x08, J8 Screw_Terminal_01x04, J9 Conn_02x04_Odd_Even, SW1 SW_Push, U1 P82B96, U10 LM2596S-ADJ, U11 RS485, U12 PC817X2NIP0F, U13 PC817X2NIP0F, U14 PC817X2NIP0F, U15 PC817X2NIP0F, U16 PC817X2NIP0F, U17 PC817X2NIP0F, U18 PC817X2NIP0F, U19 PC817X2NIP0F, U2 PC817X2NIP0F, U20 PC817X2NIP0F, U21 PC817X2NIP0F, U22 PC817X2NIP0F, U23 PC817X2NIP0F, U24 PC817X2NIP0F, U25 PC817X2NIP0F, U26 PC817X2NIP0F, U27 PC817X2NIP0F, U28 PC817X2NIP0F, U29 PC817X2NIP0F, U3 PC817X2NIP0F, U30 PC817X2NIP0F, U31 PC817X2NIP0F, U32 PC817X2NIP0F, U33 PC817X2NIP0F, U34 PC817X2NIP0F, U35 PC817X2NIP0F, U36 DS1307Z+, U37 PC817X2NIP0F, U38 PC817X2NIP0F, U39 PC817X2NIP0F, U4 PC817X2NIP0F, U40 PC817X2NIP0F, U41 PC817X2NIP0F, U42 PC817X2NIP0F, U43 PC817X2NIP0F, U44 PC817X2NIP0F, U45 PC817X2NIP0F, U46 PC817X2NIP0F, U47 PC817X2NIP0F, U48 PC817X2NIP0F, U49 PC817X2NIP0F, U5 PC817X2NIP0F, U50 PC817X2NIP0F, U51 PC817X2NIP0F, U52 PC817X2NIP0F, U53 PC817X2NIP0F, U54 PC817X2NIP0F, U55 PC817X2NIP0F, U56 PC817X2NIP0F, U6 PC817X2NIP0F, U7 PC817X2NIP0F, U8 PC817X2NIP0F, U9 PC817X2NIP0F, Y1 32,788 MHz

Commit message: correcting the scheme
Connections:
- net GND is gone; now on net Earth: BT1.2 (-), C1.2, C10.2, C11.2, C14.2, C15.2, C16.2, C17.2, C18.2, C19.2, C20.2, C21.2, C22.2, C23.2, C24.2, C25.2, C26.2, C27.2, C28.2, C29.2, C30.2, C31.2, C32.2, C33.2, C34.2, C35.2, C36.2, C37.2, C38.2, C39.2, C4.2, C40.2, C41.2, C42.2, C43.2, C44.2, C45.2, C46.2, C47.2, C48.2, C49.2, C5.2, C50.2, C51.2, C52.2, C53.2, C54.2, C55.2, C56.2, C57.2, C58.2, C6.2, C7.2, C8.2, C9.2, D2.3, I2C1.2 (Pin_2), J10.3 (Pin_3), J13.1 (Pin_1), J15.1 (Pin_1), J15.2 (Pin_2), J15.43 (Pin_43), J15.44 (Pin_44), J15.45 (Pin_45), J15.46 (Pin_46), J16.1 (Pin_1), J16.2 (Pin_2), J9.2 (Pin_2), J9.4 (Pin_4), J9.6 (Pin_6), L2.2, R38.2, U1.4 (GND), U11.4 (GND), U12.3, U13.3, U14.3, U15.3, U16.3, U17.3, U18.3, U19.3, U2.3, U20.3, U21.3, U22.3, U23.3, U24.3, U25.3, U26.3, U27.3, U28.3, U29.3, U3.3, U30.3, U31.3, U32.3, U33.3, U34.3, U35.3, U36.4 (GND), U37.3, U38.3, U39.3, U4.3, U40.3, U41.3, U42.3, U43.3, U44.3, U45.3, U46.3, U47.3, U48.3, U49.3, U5.3, U50.3, U51.3, U52.3, U53.3, U54.3, U55.3, U56.3, U6.3, U7.3, U8.3, U9.3
- net GND1 is gone; now on net Earth: J13.3 (Pin_3), J14.1 (Pin_1)
- net GNDA is gone; now on net Earth: J13.2 (Pin_2), U12.2, U13.2, U14.2, U15.2, U16.2, U17.2, U18.2, U19.2, U2.2, U20.2, U21.2, U22.2, U23.2, U24.2, U25.2, U26.2, U27.2, U28.2, U29.2, U3.2, U30.2, U31.2, U32.2, U33.2, U34.2, U35.2, U37.2, U38.2, U39.2, U4.2, U40.2, U41.2, U42.2, U43.2, U44.2, U45.2, U46.2, U47.2, U48.2, U49.2, U5.2, U50.2, U51.2, U52.2, U53.2, U54.2, U55.2, U56.2, U6.2, U7.2, U8.2, U9.2
- net GNDD is gone; now on net Earth: J10.8 (Pin_8), U11.7 (EARTH)
- net P8.03: no longer names the net of J16.3 (Pin_3)
- net P8.04: no longer names the net of J16.4 (Pin_4)
- net P8.05: no longer names the net of J16.5 (Pin_5)
- net P8.06: no longer names the net of J16.6 (Pin_6)
- net P8.20: no longer names the net of J16.20 (Pin_20)
- net P8.21: no longer names the net of J16.21 (Pin_21)
- net P8.22: no longer names the net of J16.22 (Pin_22)
- net P8.23: no longer names the net of J16.23 (Pin_23)
- net P8.24: no longer names the net of J16.24 (Pin_24)
- net P8.25: no longer names the net of J16.25 (Pin_25)
- no-connect marks 1 -> 15
