File: Circuit/boneIO - relay board 24x16A/boneIO - relay board.sch (KiCad schematic (older format))
At the start: 67 parts, among them J1 Screw_Terminal_01x04, J10 Screw_Terminal_01x04, J11 Screw_Terminal_01x04, J12 Screw_Terminal_01x04, J13 Screw_Terminal_01x04, J2 Screw_Terminal_01x04, J3 Conn_02x04_Odd_Even, J4 Screw_Terminal_01x04, J5 Screw_Terminal_01x04, J6 Screw_Terminal_01x04, J7 Screw_Terminal_01x04, J8 Screw_Terminal_01x04, J9 Screw_Terminal_01x04, K1 RM85-2011-35-1005, K10 RM85-2011-35-1005, K11 RM85-2011-35-1005, K12 RM85-2011-35-1005, K13 RM85-2011-35-1005, K14 RM85-2011-35-1005, K15 RM85-2011-35-1005, K16 RM85-2011-35-1005, K17 RM85-2011-35-1005, K18 RM85-2011-35-1005, K19 RM85-2011-35-1005, K2 RM85-2011-35-1005, K20 RM85-2011-35-1005, K21 RM85-2011-35-1005, K22 RM85-2011-35-1005, K23 RM85-2011-35-1005, K24 RM85-2011-35-1005, K3 RM85-2011-35-1005, K4 RM85-2011-35-1005, K5 RM85-2011-35-1005, K6 RM85-2011-35-1005, K7 RM85-2011-35-1005, K8 RM85-2011-35-1005, K9 RM85-2011-35-1005, SW1 SW_DIP_x03, SW2 SW_DIP_x03, SW3 SW_DIP_x03, U1 MCP9808_MSOP, U2 MCP23017_SS, U3 MCP23017_SS, U4 ULN2803A, U5 ULN2803A, U6 ULN2803A

Commit message: Correction
Corrected relay symbol on RM85-2011-35-1024
Parts:
- K1, K10, K11, K12, K13, K14, K15, K16, K17, K18, K19, K2, K20, K21, K22, K23, K24, K3, K4, K5, K6, K7, K8, K9: value RM85-2011-35-1005 -> RM85-2011-35-1024
Changed lines of the file:
@@
 P 18050 9900
 F 0 "K18" H 18700 10165 50  0000 C CNN
-F 1 "RM85-2011-35-1005" H 18700 10074 50  0000 C CNN
+F 1 "RM85-2011-35-1024" H 18700 10074 50  0000 C CNN
 F 2 "boneIO - RM85:RM852011351005_1" H 19200 10000 50  0001 L CNN
 F 3 "https://www.tme.eu/Document/59558cd216efa4c8744bca8622313f6c/e_RM85.pdf" H 19200 9900 50  0001 L CNN
@@
 P 18050 8150
 F 0 "K17" H 18700 8415 50  0000 C CNN
-F 1 "RM85-2011-35-1005" H 18700 8324 50  0000 C CNN
+F 1 "RM85-2011-35-1024" H 18700 8324 50  0000 C CNN
 F 2 "boneIO - RM85:RM852011351005_1" H 19200 8250 50  0001 L CNN
 F 3 "https://www.tme.eu/Document/59558cd216efa4c8744bca8622313f6c/e_RM85.pdf" H 19200 8150 50  0001 L CNN
@@
 P 18050 13450
 F 0 "K20" H 18700 13715 50  0000 C CNN
-F 1 "RM85-2011-35-1005" H 18700 13624 50  0000 C CNN
+F 1 "RM85-2011-35-1024" H 18700 13624 50  0000 C CNN
 F 2 "boneIO - RM85:RM852011351005_1" H 19200 13550 50  0001 L CNN
 F 3 "https://www.tme.eu/Document/59558cd216efa4c8744bca8622313f6c/e_RM85.pdf" H 19200 13450 50  0001 L CNN
@@
 P 18050 11700
 F 0 "K19" H 18700 11965 50  0000 C CNN
-F 1 "RM85-2011-35-1005" H 18700 11874 50  0000 C CNN
+F 1 "RM85-2011-35-1024" H 18700 11874 50  0000 C CNN
 F 2 "boneIO - RM85:RM852011351005_1" H 19200 11800 50  0001 L CNN
 F 3 "https://www.tme.eu/Document/59558cd216efa4c8744bca8622313f6c/e_RM85.pdf" H 19200 11700 50  0001 L CNN
@@
 P 13300 9900
 F 0 "K14" H 13950 10165 50  0000 C CNN
-F 1 "RM85-2011-35-1005" H 13950 10074 50  0000 C CNN
+F 1 "RM85-2011-35-1024" H 13950 10074 50  0000 C CNN
 F 2 "boneIO - RM85:RM852011351005_1" H 14450 10000 50  0001 L CNN
 F 3 "https://www.tme.eu/Document/59558cd216efa4c8744bca8622313f6c/e_RM85.pdf" H 14450 9900 50  0001 L CNN
@@
 P 13300 8150
 F 0 "K13" H 13950 8415 50  0000 C CNN
-F 1 "RM85-2011-35-1005" H 13950 8324 50  0000 C CNN
+F 1 "RM85-2011-35-1024" H 13950 8324 50  0000 C CNN
 F 2 "boneIO - RM85:RM852011351005_1" H 14450 8250 50  0001 L CNN
 F 3 "https://www.tme.eu/Document/59558cd216efa4c8744bca8622313f6c/e_RM85.pdf" H 14450 8150 50  0001 L CNN
@@
 P 13300 13450
 F 0 "K16" H 13950 13715 50  0000 C CNN
-F 1 "RM85-2011-35-1005" H 13950 13624 50  0000 C CNN
+F 1 "RM85-2011-35-1024" H 13950 13624 50  0000 C CNN
 F 2 "boneIO - RM85:RM852011351005_1" H 14450 13550 50  0001 L CNN
 F 3 "https://www.tme.eu/Document/59558cd216efa4c8744bca8622313f6c/e_RM85.pdf" H 14450 13450 50  0001 L CNN
@@
 P 13300 11700
 F 0 "K15" H 13950 11965 50  0000 C CNN
-F 1 "RM85-2011-35-1005" H 13950 11874 50  0000 C CNN
+F 1 "RM85-2011-35-1024" H 13950 11874 50  0000 C CNN
 F 2 "boneIO - RM85:RM852011351005_1" H 14450 11800 50  0001 L CNN
 F 3 "https://www.tme.eu/Document/59558cd216efa4c8744bca8622313f6c/e_RM85.pdf" H 14450 11700 50  0001 L CNN
@@
 P 10800 11700
 F 0 "K11" H 11450 11965 50  0000 C CNN
-F 1 "RM85-2011-35-1005" H 11450 11874 50  0000 C CNN
+F 1 "RM85-2011-35-1024" H 11450 11874 50  0000 C CNN
 F 2 "boneIO - RM85:RM852011351005_1" H 11950 11800 50  0001 L CNN
 F 3 "https://www.tme.eu/Document/59558cd216efa4c8744bca8622313f6c/e_RM85.pdf" H 11950 11700 50  0001 L CNN
@@
 P 10800 13450
 F 0 "K12" H 11450 13715 50  0000 C CNN
-F 1 "RM85-2011-35-1005" H 11450 13624 50  0000 C CNN
+F 1 "RM85-2011-35-1024" H 11450 13624 50  0000 C CNN
 F 2 "boneIO - RM85:RM852011351005_1" H 11950 13550 50  0001 L CNN
 F 3 "https://www.tme.eu/Document/59558cd216efa4c8744bca8622313f6c/e_RM85.pdf" H 11950 13450 50  0001 L CNN
@@
 P 10800 8150
 F 0 "K9" H 11450 8415 50  0000 C CNN
-F 1 "RM85-2011-35-1005" H 11450 8324 50  0000 C CNN
+F 1 "RM85-2011-35-1024" H 11450 8324 50  0000 C CNN
 F 2 "boneIO - RM85:RM852011351005_1" H 11950 8250 50  0001 L CNN
 F 3 "https://www.tme.eu/Document/59558cd216efa4c8744bca8622313f6c/e_RM85.pdf" H 11950 8150 50  0001 L CNN
@@
 P 10800 9900
 F 0 "K10" H 11450 10165 50  0000 C CNN
-F 1 "RM85-2011-35-1005" H 11450 10074 50  0000 C CNN
+F 1 "RM85-2011-35-1024" H 11450 10074 50  0000 C CNN
 F 2 "boneIO - RM85:RM852011351005_1" H 11950 10000 50  0001 L CNN
 F 3 "https://www.tme.eu/Document/59558cd216efa4c8744bca8622313f6c/e_RM85.pdf" H 11950 9900 50  0001 L CNN
@@
 P 6100 9900
 F 0 "K6" H 6750 10165 50  0000 C CNN
-F 1 "RM85-2011-35-1005" H 6750 10074 50  0000 C CNN
+F 1 "RM85-2011-35-1024" H 6750 10074 50  0000 C CNN
 F 2 "boneIO - RM85:RM852011351005_1" H 7250 10000 50  0001 L CNN
 F 3 "https://www.tme.eu/Document/59558cd216efa4c8744bca8622313f6c/e_RM85.pdf" H 7250 9900 50  0001 L CNN
@@
 P 6100 8150
 F 0 "K5" H 6750 8415 50  0000 C CNN
-F 1 "RM85-2011-35-1005" H 6750 8324 50  0000 C CNN
+F 1 "RM85-2011-35-1024" H 6750 8324 50  0000 C CNN
 F 2 "boneIO - RM85:RM852011351005_1" H 7250 8250 50  0001 L CNN
 F 3 "https://www.tme.eu/Document/59558cd216efa4c8744bca8622313f6c/e_RM85.pdf" H 7250 8150 50  0001 L CNN
@@
 P 6100 13450
 F 0 "K8" H 6750 13715 50  0000 C CNN
-F 1 "RM85-2011-35-1005" H 6750 13624 50  0000 C CNN
+F 1 "RM85-2011-35-1024" H 6750 13624 50  0000 C CNN
 F 2 "boneIO - RM85:RM852011351005_1" H 7250 13550 50  0001 L CNN
 F 3 "https://www.tme.eu/Document/59558cd216efa4c8744bca8622313f6c/e_RM85.pdf" H 7250 13450 50  0001 L CNN
@@
 P 6100 11700
 F 0 "K7" H 6750 11965 50  0000 C CNN
-F 1 "RM85-2011-35-1005" H 6750 11874 50  0000 C CNN
+F 1 "RM85-2011-35-1024" H 6750 11874 50  0000 C CNN
 F 2 "boneIO - RM85:RM852011351005_1" H 7250 11800 50  0001 L CNN
 F 3 "https://www.tme.eu/Document/59558cd216efa4c8744bca8622313f6c/e_RM85.pdf" H 7250 11700 50  0001 L CNN
@@
 P 3600 11700
 F 0 "K3" H 4250 11965 50  0000 C CNN
-F 1 "RM85-2011-35-1005" H 4250 11874 50  0000 C CNN
+F 1 "RM85-2011-35-1024" H 4250 11874 50  0000 C CNN
 F 2 "boneIO - RM85:RM852011351005_1" H 4750 11800 50  0001 L CNN
 F 3 "https://www.tme.eu/Document/59558cd216efa4c8744bca8622313f6c/e_RM85.pdf" H 4750 11700 50  0001 L CNN
@@
 P 3600 13450
 F 0 "K4" H 4250 13715 50  0000 C CNN
-F 1 "RM85-2011-35-1005" H 4250 13624 50  0000 C CNN
+F 1 "RM85-2011-35-1024" H 4250 13624 50  0000 C CNN
 F 2 "boneIO - RM85:RM852011351005_1" H 4750 13550 50  0001 L CNN
 F 3 "https://www.tme.eu/Document/59558cd216efa4c8744bca8622313f6c/e_RM85.pdf" H 4750 13450 50  0001 L CNN
@@
 P 3600 8150
 F 0 "K1" H 4250 8415 50  0000 C CNN
-F 1 "RM85-2011-35-1005" H 4250 8324 50  0000 C CNN
+F 1 "RM85-2011-35-1024" H 4250 8324 50  0000 C CNN
 F 2 "boneIO - RM85:RM852011351005_1" H 4750 8250 50  0001 L CNN
 F 3 "https://www.tme.eu/Document/59558cd216efa4c8744bca8622313f6c/e_RM85.pdf" H 4750 8150 50  0001 L CNN
@@
 P 3600 9900
 F 0 "K2" H 4250 10165 50  0000 C CNN
-F 1 "RM85-2011-35-1005" H 4250 10074 50  0000 C CNN
+F 1 "RM85-2011-35-1024" H 4250 10074 50  0000 C CNN
 F 2 "boneIO - RM85:RM852011351005_1" H 4750 10000 50  0001 L CNN
 F 3 "https://www.tme.eu/Document/59558cd216efa4c8744bca8622313f6c/e_RM85.pdf" H 4750 9900 50  0001 L CNN
@@
 P 21200 11700
 F 0 "K23" H 21850 11965 50  0000 C CNN
-F 1 "RM85-2011-35-1005" H 21850 11874 50  0000 C CNN
+F 1 "RM85-2011-35-1024" H 21850 11874 50  0000 C CNN
 F 2 "boneIO - RM85:RM852011351005_1" H 22350 11800 50  0001 L CNN
 F 3 "https://www.tme.eu/Document/59558cd216efa4c8744bca8622313f6c/e_RM85.pdf" H 22350 11700 50  0001 L CNN
@@
 P 21200 13450
 F 0 "K24" H 21850 13715 50  0000 C CNN
-F 1 "RM85-2011-35-1005" H 21850 13624 50  0000 C CNN
+F 1 "RM85-2011-35-1024" H 21850 13624 50  0000 C CNN
 F 2 "boneIO - RM85:RM852011351005_1" H 22350 13550 50  0001 L CNN
 F 3 "https://www.tme.eu/Document/59558cd216efa4c8744bca8622313f6c/e_RM85.pdf" H 22350 13450 50  0001 L CNN
@@
 P 21200 8150
 F 0 "K21" H 21850 8415 50  0000 C CNN
-F 1 "RM85-2011-35-1005" H 21850 8324 50  0000 C CNN
+F 1 "RM85-2011-35-1024" H 21850 8324 50  0000 C CNN
 F 2 "boneIO - RM85:RM852011351005_1" H 22350 8250 50  0001 L CNN
 F 3 "https://www.tme.eu/Document/59558cd216efa4c8744bca8622313f6c/e_RM85.pdf" H 22350 8150 50  0001 L CNN
@@
 P 21200 9900
 F 0 "K22" H 21850 10165 50  0000 C CNN
-F 1 "RM85-2011-35-1005" H 21850 10074 50  0000 C CNN
+F 1 "RM85-2011-35-1024" H 21850 10074 50  0000 C CNN
 F 2 "boneIO - RM85:RM852011351005_1" H 22350 10000 50  0001 L CNN
 F 3 "https://www.tme.eu/Document/59558cd216efa4c8744bca8622313f6c/e_RM85.pdf" H 22350 9900 50  0001 L CNN

Commit message: correcting the scheme
Changed lines of the file:
@@
 Wire Wire Line
 	18050 13550 18250 13550
-Text Notes 6100 2400 0    197  ~ 39
+Text Notes 5200 2200 0    197  ~ 39
 PINOUT
 Text Notes 11500 2350 0    197  ~ 39
@@
 	21700 2250 21700 2500
 Connection ~ 21700 2500
+$Comp
+L power:PWR_FLAG #FLG0101
+U 1 1 619EE2AC
+P 7150 2200
+F 0 "#FLG0101" H 7150 2275 50  0001 C CNN
+F 1 "PWR_FLAG" H 7150 2373 50  0000 C CNN
+F 2 "" H 7150 2200 50  0001 C CNN
+F 3 "~" H 7150 2200 50  0001 C CNN
+	1    7150 2200
+	-1   0    0    1
+$EndComp
+$Comp
+L power:+3V3 #PWR0133
+U 1 1 619EE9F3
+P 7150 2050
+F 0 "#PWR0133" H 7150 1900 50  0001 C CNN
+F 1 "+3V3" H 7165 2223 50  0000 C CNN
+F 2 "" H 7150 2050 50  0001 C CNN
+F 3 "" H 7150 2050 50  0001 C CNN
+	1    7150 2050
+	1    0    0    -1
+$EndComp
+Wire Wire Line
+	7150 2200 7150 2050
+$Comp
+L power:+5V #PWR0134
+U 1 1 61AA15B4
+P 7400 2050
+F 0 "#PWR0134" H 7400 1900 50  0001 C CNN
+F 1 "+5V" H 7415 2223 50  0000 C CNN
+F 2 "" H 7400 2050 50  0001 C CNN
+F 3 "" H 7400 2050 50  0001 C CNN
+	1    7400 2050
+	1    0    0    -1
+$EndComp
+$Comp
+L power:PWR_FLAG #FLG0102
+U 1 1 61ADCEBD
+P 7400 2200
+F 0 "#FLG0102" H 7400 2275 50  0001 C CNN
+F 1 "PWR_FLAG" H 7400 2373 50  0000 C CNN
+F 2 "" H 7400 2200 50  0001 C CNN
+F 3 "~" H 7400 2200 50  0001 C CNN
+	1    7400 2200
+	-1   0    0    1
+$EndComp
+Wire Wire Line
+	7400 2200 7400 2050
+$Comp
+L power:+24V #PWR0135
+U 1 1 61B18DCF
+P 7700 2050
+F 0 "#PWR0135" H 7700 1900 50  0001 C CNN
+F 1 "+24V" H 7715 2223 50  0000 C CNN
+F 2 "" H 7700 2050 50  0001 C CNN
+F 3 "" H 7700 2050 50  0001 C CNN
+	1    7700 2050
+	1    0    0    -1
+$EndComp
+$Comp
+L power:PWR_FLAG #FLG0103
+U 1 1 61B54C9F
+P 7700 2200
+F 0 "#FLG0103" H 7700 2275 50  0001 C CNN
+F 1 "PWR_FLAG" H 7700 2373 50  0000 C CNN
+F 2 "" H 7700 2200 50  0001 C CNN
+F 3 "~" H 7700 2200 50  0001 C CNN
+	1    7700 2200
+	-1   0    0    1
+$EndComp
+Wire Wire Line
+	7700 2200 7700 2050
+$Comp
+L power:GND #PWR0136
+U 1 1 61BCD558
+P 8000 2050
+F 0 "#PWR0136" H 8000 1800 50  0001 C CNN
+F 1 "GND" H 8005 1877 50  0000 C CNN
+F 2 "" H 8000 2050 50  0001 C CNN
+F 3 "" H 8000 2050 50  0001 C CNN
+	1    8000 2050
+	-1   0    0    1
+$EndComp
+Wire Wire Line
+	8000 2200 8000 2050
+$Comp
+L power:VCC #PWR0137
+U 1 1 61CFBC73
+P 6900 2050
+F 0 "#PWR0137" H 6900 1900 50  0001 C CNN
+F 1 "VCC" H 6915 2223 50  0000 C CNN
+F 2 "" H 6900 2050 50  0001 C CNN
+F 3 "" H 6900 2050 50  0001 C CNN
+	1    6900 2050
+	1    0    0    -1
+$EndComp
+$Comp
+L power:PWR_FLAG #FLG0104
+U 1 1 61D38686
+P 6900 2200
+F 0 "#FLG0104" H 6900 2275 50  0001 C CNN
+F 1 "PWR_FLAG" H 6900 2373 50  0000 C CNN
+F 2 "" H 6900 2200 50  0001 C CNN
+F 3 "~" H 6900 2200 50  0001 C CNN
+	1    6900 2200
+	-1   0    0    1
+$EndComp
+Wire Wire Line
+	6900 2200 6900 2050
+$Comp
+L power:PWR_FLAG #FLG0105
+U 1 1 61DB26DF
+P 8000 2200
+F 0 "#FLG0105" H 8000 2275 50  0001 C CNN
+F 1 "PWR_FLAG" H 8000 2373 50  0000 C CNN
+F 2 "" H 8000 2200 50  0001 C CNN
+F 3 "~" H 8000 2200 50  0001 C CNN
+	1    8000 2200
+	-1   0    0    1
+$EndComp
 $EndSCHEMATC
